File: AD1868I2S.kicad_sch (KiCad schematic)
At the start: 16 parts, among them J1 054986, J2 JTAG, J3 I2S, SW1 MODE, U1 EPM3064A(TQFP), U2 AMS1117-3.3, X1 22.5792MHz

Commit message: update pcb to rev2
Parts:
- removed R1, R2: 10k, Resistor_SMD:R_0603_1608Metric_Pad0.98x0.95mm_HandSolder, symbol Device:R
- removed SW1: MODE, Button_Switch_THT:SW_DIP_SPSTx02_Slide_9.78x7.26mm_W7.62mm_P2.54mm, symbol Switch:SW_DIP_x02
- added J4: Conn_01x03, Jumper:SolderJumper-3_P1.3mm_Open_Pad1.0x1.5mm, symbol Connector_Generic:Conn_01x03
- added U3: 74HC86, Package_SO:SOIC-14_3.9x8.7mm_P1.27mm, symbol 74xx:74HC86
Connections:
- net +3.3V: now also U3.1, U3.14 (VCC)
- net GND: now also U3.10, U3.12, U3.13, U3.4, U3.5, U3.7 (GND), U3.9
- net I2S_MCK: now also J4.2 (Pin_2); no longer C5.1, X1.3 (OUT)
- net DIP1: no longer names the net of U1.8 (I/O)
- net DIP2: no longer names the net of U1.10 (I/O)
- new net XCK: C5.1, J4.1 (Pin_1), U3.2, X1.3 (OUT)
- new net XCK_X: J4.3 (Pin_3), U3.3
- no-connect marks 27 -> 29
Other:
- note removed: "X1 - wrong footprint layout correct: 4 3 1 2"
- moved on the sheet: C5, X1

Commit message: rev3
Parts:
- added C10, C11, C8, C9: 0.1uF, Capacitor_SMD:C_0603_1608Metric_Pad1.08x0.95mm_HandSolder, symbol Device:C
- added U4: EPM3064A(TQFP), Package_QFP:TQFP-44_10x10mm_P0.8mm, symbol toyoshim:EPM3064A(TQFP)
Connections:
- net +3.3V: now also C10.1, C11.1, C8.1, C9.1, U4.17 (VCC), U4.29 (VCC), U4.41 (VCC), U4.9 (VCC)
- net CK: now also U1.42 (I/O); no longer U1.40 (INPUT/OE2/GCLK2)
- net DL: now also U4.40 (INPUT/OE2/GCLK2); no longer U1.35 (I/O)
- net DR: now also U1.40 (INPUT/OE2/GCLK2); no longer U1.43 (I/O)
- net GND: now also C10.2, C11.2, C8.2, C9.2, U4.11 (GND), U4.16 (GND), U4.24 (GND), U4.30 (GND), U4.36 (GND), U4.4 (GND)
- net I2S_CLK: now also U1.44 (I/O), U4.42 (I/O); no longer U1.2 (I/O)
- net I2S_DT: now also U4.33 (I/O); no longer U1.3 (I/O)
- net I2S_LR: now also U4.31 (I/O); no longer U1.5 (I/O)
- net LL: no longer U1.42 (I/O)
- net LR: now also U1.35 (I/O); no longer U1.44 (I/O)
- net TCK: now also U4.26 (I/O/TCK)
- net TDO: now also U4.32 (I/O/TDO); no longer U1.32 (I/O/TDO)
- net TMS: now also U4.7 (I/O/TMS)
- net DR3: now reaches U1.10 (I/O)
- net DR3: now also U4.23 (I/O)
- net DR4: now reaches U1.12 (I/O)
- net DR4: now also U4.22 (I/O)
- net DR5: now reaches U1.13 (I/O)
- net DR5: now also U4.21 (I/O)
- net DR6: now reaches U1.14 (I/O)
- net DR6: now also U4.20 (I/O)
- net DR7: now reaches U1.15 (I/O)
- net DR7: now also U4.19 (I/O)
- net DR8: now reaches U1.18 (I/O)
- net DR8: now also U4.18 (I/O)
- net DR9: now reaches U1.19 (I/O)
- net DR9: now also U4.15 (I/O)
- net DR10: now reaches U1.20 (I/O)
- net DR10: now also U4.14 (I/O)
- net DR11: now reaches U1.21 (I/O)
- net DR11: now also U4.13 (I/O)
- net DR12: now reaches U1.22 (I/O)
- net DR12: now also U4.12 (I/O)
- net DR13: now reaches U1.23 (I/O)
- net DR13: now also U4.10 (I/O)
- net DR14: now reaches U1.25 (I/O)
- net DR14: now also U4.8 (I/O)
- net DR15: now reaches U1.27 (I/O)
- net DR15: now also U4.6 (I/O)
- net DR16: now reaches U1.28 (I/O)
- net DR16: now also U4.5 (I/O)
- net DR17: now reaches U1.31 (I/O)
- net DR17: now also U4.3 (I/O)
- net AD_LP: now reaches U1.33 (I/O)
- net AD_LP: now also U4.2 (I/O)
- net LATCH: now reaches U1.34 (I/O)
- net LATCH: now also U4.44 (I/O)
- net DR1: now reaches U1.6 (I/O)
- net DR1: now also U4.27 (I/O)
- net DR2: now reaches U1.8 (I/O)
- net DR2: now also U4.25 (I/O)
- new net DR0: U1.5 (I/O), U4.28 (I/O)
- new net SYNC_CLK: U1.43 (I/O), U4.43 (I/O)
- new net TDX: U1.32 (I/O/TDO), U4.1 (I/O/TDI)
- no-connect marks 29 -> 20
Other:
- moved on the sheet: C1, C2, C3, C4, J3, U1
